Commit message: feat: working gazebo/rviz sim of jackal

File: src/catkin_ws/src/jackal_custom/urdf/xacro/jackal.gazebo.xacro (robot description, xacro)
@@ -9,5 +9,5 @@
     <plugin name="imu_controller" filename="libhector_gazebo_ros_imu.so">
       <!-- <robotNamespace>/</robotNamespace> -->
-      <updateRate>50.0</updateRate>
+      <updateRate>10.0</updateRate>
       <bodyName>imu_link</bodyName>
       <topicName>imu/data</topicName>
@@ -42,5 +42,5 @@
     <turnGravityOff>false</turnGravityOff>
   </gazebo>
-    <gazebo reference="imu_link">
+  <gazebo reference="imu_link">
     <turnGravityOff>false</turnGravityOff>
   </gazebo>

File: src/catkin_ws/src/jackal_custom/urdf/xacro/jackal_custom.urdf.xacro (robot description, xacro)
@@ -1,17 +1,9 @@
 <?xml version="1.0"?>
 <robot xmlns:xacro="http://www.ros.org/wiki/xacro" name="Jackal">
-    <xacro:include filename="$(find jackal_custom)/urdf/custom_jackal_base.urdf.xacro" />
-    <xacro:arg name="rear_id" default="0" />
+    <xacro:include filename="$(find jackal_custom)/urdf/xacro/jackal_custom_base.urdf.xacro" />
     <xacro:arg name="right_id" default="1" />
     <xacro:arg name="left_id" default="2" />
-    <xacro:property name="rear" value="$(arg rear_id)" />
     <xacro:property name="right" value="$(arg right_id)" />
     <xacro:property name="left" value="$(arg left_id)" />
-    <link name="vicon_link"></link>
-    <joint name="vicon_link_joint" type="fixed">
-      <origin xyz="0.085 0 0.184" rpy="0 0 0" />
-      <parent link="base_link"/>
-      <child link="vicon_link" />
-    </joint>
     <!-- -->
     <link name="right_tag">
@@ -46,5 +38,5 @@
     </gazebo>
     <gazebo reference="right_tag">
-        <material>Gazebo/White</material>
+        <material>Gazebo/Green</material>
     </gazebo>
     <!-- -->
@@ -80,39 +72,5 @@
     </gazebo>
     <gazebo reference="left_tag">
-        <material>Gazebo/White</material>
-    </gazebo>
-    <!-- -->
-    <link name="rear_tag">
-        <inertial>
-            <mass value="0.1" />
-            <origin rpy="0 0 0" xyz="0 0 0"/>
-            <inertia ixx="1.0" ixy="0.0" ixz="0.0" iyy="1.0" iyz="0.0" izz="1.0" />
-        </inertial>
-        <collision>
-            <origin xyz="0 -0.013 0" rpy="0 0 0"/>
-            <geometry>
-                <box size="0.05 0.026 0.102"/>
-            </geometry>
-        </collision>
-        <visual>
-            <origin xyz="0 0 0" rpy="-1.57 0 -1.57"/>
-            <geometry>
-                <mesh filename="package://jackal_custom/models/DecaWave/meshes/Decawave.stl"/>
-            </geometry>
-            <!--material name="rear_tag_color">
-                <color rgba="0 0 200 0"/>
-            </material-->
-        </visual>
-    </link>
-    <joint name="rear_tag_joint" type="fixed">
-        <origin xyz="-0.19 0.0 0.184" rpy="0 0 0"/>
-        <parent link="chassis_link"/>
-        <child link="rear_tag"/>
-    </joint>
-    <gazebo reference="rear_tag_joint">
-        <preserveFixedJoint>true</preserveFixedJoint>
-    </gazebo>
-    <gazebo reference="rear_tag">
-        <material>Gazebo/White</material>
+        <material>Gazebo/Red</material>
     </gazebo>
 </robot>

File: src/catkin_ws/src/jackal_custom/urdf/xacro/jackal_custom_base.urdf.xacro (robot description, xacro)
@@ -68,16 +68,16 @@
     </transmission>
   </xacro:macro>
-  <link name="world"></link>
-  <joint name="world_joint" type="fixed">
-    <origin xyz="0 0 0" rpy="0 0 0" />
-    <parent link="world"/>
-    <child link="world" />
-  </joint>
-  <link name="odom"></link>
-  <joint name="odom_joint" type="fixed">
-    <origin xyz="0 0 0" rpy="0 0 0" />
-    <parent link="odom"/>
-    <child link="base_link" />
-  </joint>
+  <xacro:wheel prefix="front_left">
+    <origin xyz="${wheelbase/2} ${track/2} ${wheel_vertical_offset}" rpy="0 0 0" />
+  </xacro:wheel>
+  <xacro:wheel prefix="front_right">
+    <origin xyz="${wheelbase/2} ${-track/2} ${wheel_vertical_offset}" rpy="0 0 0" />
+  </xacro:wheel>
+  <xacro:wheel prefix="rear_left">
+    <origin xyz="${-wheelbase/2} ${track/2} ${wheel_vertical_offset}" rpy="0 0 0" />
+  </xacro:wheel>
+  <xacro:wheel prefix="rear_right">
+    <origin xyz="${-wheelbase/2} ${-track/2} ${wheel_vertical_offset}" rpy="0 0 0" />
+  </xacro:wheel>
   <link name="base_link"></link>
   <joint name="base_link_joint" type="fixed">
@@ -111,16 +111,4 @@
       </inertial>
   </link>
-  <xacro:wheel prefix="front_left">
-    <origin xyz="${wheelbase/2} ${track/2} ${wheel_vertical_offset}" rpy="0 0 0" />
-  </xacro:wheel>
-  <xacro:wheel prefix="front_right">
-    <origin xyz="${wheelbase/2} ${-track/2} ${wheel_vertical_offset}" rpy="0 0 0" />
-  </xacro:wheel>
-  <xacro:wheel prefix="rear_left">
-    <origin xyz="${-wheelbase/2} ${track/2} ${wheel_vertical_offset}" rpy="0 0 0" />
-  </xacro:wheel>
-  <xacro:wheel prefix="rear_right">
-    <origin xyz="${-wheelbase/2} ${-track/2} ${wheel_vertical_offset}" rpy="0 0 0" />
-  </xacro:wheel>
   <xacro:unless value="$(optenv JACKAL_FRONT_ACCESSORY_FENDER 0)">
     <link name="front_fender_link">
@@ -232,16 +220,14 @@
   </joint>
   <!-- Bring in simulation data for Gazebo. -->
-  <xacro:include filename="$(find jackal_custom)/urdf/jackal.gazebo" />
+  <xacro:include filename="$(find jackal_custom)/urdf/xacro/jackal.gazebo.xacro" />
   <!-- Optional standard accessories, including their simulation data. The rendering
        of these into the final description is controlled by optenv variables, which
        default each one to off.-->
   <!--xacro:include filename="$(find jackal_description)/urdf/accessories.urdf.xacro" /-->
-  <!-- Optional custom includes. -->
-  <xacro:include filename="$(optenv JACKAL_URDF_EXTRAS empty.urdf)" />
   <!---->
   <gazebo>
       <plugin name="p3d_base_controller" filename="libgazebo_ros_p3d.so">
           <alwaysOn>true</alwaysOn>
-          <updateRate>50.0</updateRate>
+          <updateRate>10.0</updateRate>
           <bodyName>odom</bodyName>
           <frameName>world</frameName>
