Commit message: dev: unify the launch files

File: src/catkin_ws/src/jackal_custom/urdf/xacro/jackal_custom_base_real.urdf.xacro (robot description, xacro)
@@ -56,13 +56,4 @@
       </inertial>
     </link>
-    <gazebo reference="${prefix}_wheel_link">
-      <material>Gazebo/DarkGrey</material>
-      <selfCollide>false</selfCollide>
-      <mu1 value="1"/>
-      <mu2 value="1"/>
-      <kp value="10000000.0" />
-      <kd value="1" />
-      <fdir1 value="1 0 0"/>
-    </gazebo>
     <joint name="${prefix}_wheel" type="continuous">
       <parent link="$(arg ns)chassis_link"/>

Commit message: dev: try to fix wheels

File: src/catkin_ws/src/jackal_custom/urdf/xacro/jackal_custom_base_real.urdf.xacro (robot description, xacro)
@@ -62,4 +62,16 @@
       <axis xyz="0 1 0" />
     </joint>
+    <!-- In reality, Jackal has only two motors, one per side. However, it's more
+        straightforward for Gazebo to simulate as if there's an actuator per wheel.
+        So we keep it also in the real one. -->
+    <transmission name="${prefix}_wheel_trans">
+      <type>transmission_interface/SimpleTransmission</type>
+      <joint name="${prefix}_wheel">
+        <hardwareInterface>hardware_interface/VelocityJointInterface</hardwareInterface>
+      </joint>
+      <actuator name="${prefix}_actuator">
+        <mechanicalReduction>1</mechanicalReduction>
+      </actuator>
+    </transmission>
   </xacro:macro>
   <xacro:wheel prefix="$(arg ns)front_left">

Commit message: dev: testing the encoder in EKF

File: src/catkin_ws/src/jackal_custom/urdf/xacro/jackal_custom_base_real.urdf.xacro (robot description, xacro)
@@ -33,4 +33,22 @@
   </material>
   <xacro:macro name="wheel" params="prefix *joint_pose">
+    <joint name="${prefix}_wheel" type="continuous">
+      <parent link="$(arg ns)chassis_link"/>
+      <child link="${prefix}_wheel_link" />
+      <xacro:insert_block name="joint_pose" />
+      <axis xyz="0 1 0" />
+    </joint>
+    <!-- In reality, Jackal has only two motors, one per side. However, it's more
+        straightforward for Gazebo to simulate as if there's an actuator per wheel.
+        So we keep it also in the real -->
+    <transmission name="${prefix}_wheel_trans">
+      <type>transmission_interface/SimpleTransmission</type>
+      <joint name="${prefix}_wheel">
+        <hardwareInterface>hardware_interface/VelocityJointInterface</hardwareInterface>
+      </joint>
+      <actuator name="${prefix}_actuator">
+        <mechanicalReduction>1</mechanicalReduction>
+      </actuator>
+    </transmission>
     <link name="${prefix}_wheel_link">
       <visual>
@@ -56,33 +74,15 @@
       </inertial>
     </link>
-    <joint name="${prefix}_wheel" type="continuous">
-      <parent link="$(arg ns)chassis_link"/>
-      <child link="${prefix}_wheel_link" />
-      <xacro:insert_block name="joint_pose" />
-      <axis xyz="0 1 0" />
-    </joint>
-    <!-- In reality, Jackal has only two motors, one per side. However, it's more
-        straightforward for Gazebo to simulate as if there's an actuator per wheel.
-        So we keep it also in the real one. -->
-    <transmission name="${prefix}_wheel_trans">
-      <type>transmission_interface/SimpleTransmission</type>
-      <joint name="${prefix}_wheel">
-        <hardwareInterface>hardware_interface/VelocityJointInterface</hardwareInterface>
-      </joint>
-      <actuator name="${prefix}_actuator">
-        <mechanicalReduction>1</mechanicalReduction>
-      </actuator>
-    </transmission>
   </xacro:macro>
-  <xacro:wheel prefix="$(arg ns)front_left">
+  <xacro:wheel prefix="front_left">
     <origin xyz="${wheelbase/2} ${track/2} ${wheel_vertical_offset}" rpy="0 0 0" />
   </xacro:wheel>
-  <xacro:wheel prefix="$(arg ns)front_right">
+  <xacro:wheel prefix="front_right">
     <origin xyz="${wheelbase/2} ${-track/2} ${wheel_vertical_offset}" rpy="0 0 0" />
   </xacro:wheel>
-  <xacro:wheel prefix="$(arg ns)rear_left">
+  <xacro:wheel prefix="rear_left">
     <origin xyz="${-wheelbase/2} ${track/2} ${wheel_vertical_offset}" rpy="0 0 0" />
   </xacro:wheel>
-  <xacro:wheel prefix="$(arg ns)rear_right">
+  <xacro:wheel prefix="rear_right">
     <origin xyz="${-wheelbase/2} ${-track/2} ${wheel_vertical_offset}" rpy="0 0 0" />
   </xacro:wheel>
