Commit message: chore: IP

File: src/catkin_ws/src/jackal_custom/urdf/xacro/jackal_custom_base.urdf.xacro (robot description, xacro)
@@ -258,5 +258,5 @@
       <parent link="$(arg ns)chassis_link"/>
       <child link="$(arg ns)right_tag"/>
-      <origin xyz="0 0 0.184" rpy="0 0 0"/>
+      <origin xyz="0.165 -0.135 0.184" rpy="0 0 0"/>
   </joint>
   <!-- Bring in simulation data for Gazebo. -->

File: src/catkin_ws/src/jackal_custom/urdf/xacro/jackal_custom_base_real.urdf.xacro (robot description, xacro)
@@ -229,10 +229,10 @@
   <link name="$(arg ns)right_tag">
       <inertial>
-          <origin xyz="0 0 0.184" rpy="-1.57 0 -1.57"/>
+          <origin xyz="0 0 0" rpy="-1.57 0 -1.57"/>
           <mass value="0.1" />
           <inertia ixx="1.0" ixy="0.0" ixz="0.0" iyy="1.0" iyz="0.0" izz="1.0" />
       </inertial>
       <collision>
-          <origin xyz="0 0 0.184" rpy="-1.57 0 -1.57"/>
+          <origin xyz="0 0 0" rpy="-1.57 0 -1.57"/>
           <geometry>
               <box size="0.05 0.026 0.102"/>
@@ -240,5 +240,5 @@
       </collision>
       <visual>
-          <origin xyz="0 0 0.184" rpy="-1.57 0 -1.57"/>
+          <origin xyz="0 0 0" rpy="-1.57 0 -1.57"/>
           <geometry>
               <mesh filename="package://jackal_custom/models/DecaWave/meshes/Decawave.stl"/>
@@ -250,4 +250,5 @@
       <parent link="$(arg ns)chassis_link"/>
       <child link="$(arg ns)right_tag"/>
+      <origin xyz="0.165 -0.135 0.184" rpy="0 0 0"/>
   </joint>
 </robot>

Commit message: feat: working gazebo/rviz sim of jackal

File: src/catkin_ws/src/jackal_custom/urdf/xacro/jackal_custom_base.urdf.xacro (robot description, xacro)
@@ -1,4 +1,10 @@
 <?xml version="1.0"?>
 <robot name="jackal" xmlns:xacro="http://www.ros.org/wiki/xacro">
+  <!-- Parameters -->
+  <xacro:arg name="right_id" default="1" />
+  <xacro:arg name="ns" default="" />
+  <xacro:property name="right" value="$(arg right_id)" />
+  <xacro:property name="ns" value="$(arg ns)" />
+  <!-- Fixed values -->
   <xacro:property name="PI" value="3.1415926535897931" />
   <xacro:property name="wheelbase" value="0.262" />
@@ -51,5 +57,5 @@
     </gazebo>
     <joint name="${prefix}_wheel" type="continuous">
-      <parent link="chassis_link"/>
+      <parent link="$(arg ns)chassis_link"/>
       <child link="${prefix}_wheel_link" />
       <xacro:insert_block name="joint_pose" />
@@ -68,23 +74,23 @@
     </transmission>
   </xacro:macro>
-  <xacro:wheel prefix="front_left">
+  <xacro:wheel prefix="$(arg ns)front_left">
     <origin xyz="${wheelbase/2} ${track/2} ${wheel_vertical_offset}" rpy="0 0 0" />
   </xacro:wheel>
-  <xacro:wheel prefix="front_right">
+  <xacro:wheel prefix="$(arg ns)front_right">
     <origin xyz="${wheelbase/2} ${-track/2} ${wheel_vertical_offset}" rpy="0 0 0" />
   </xacro:wheel>
-  <xacro:wheel prefix="rear_left">
+  <xacro:wheel prefix="$(arg ns)rear_left">
     <origin xyz="${-wheelbase/2} ${track/2} ${wheel_vertical_offset}" rpy="0 0 0" />
   </xacro:wheel>
-  <xacro:wheel prefix="rear_right">
+  <xacro:wheel prefix="$(arg ns)rear_right">
     <origin xyz="${-wheelbase/2} ${-track/2} ${wheel_vertical_offset}" rpy="0 0 0" />
   </xacro:wheel>
-  <link name="base_link"></link>
+  <link name="$(arg ns)base_link"></link>
   <joint name="base_link_joint" type="fixed">
     <origin xyz="0 0 0" rpy="0 0 0" />
-    <parent link="base_link"/>
-    <child link="chassis_link" />
-  </joint>
-  <link name="chassis_link">
+    <parent link="$(arg ns)base_link"/>
+    <child link="$(arg ns)chassis_link" />
+  </joint>
+  <link name="$(arg ns)chassis_link">
     <visual>
       <origin xyz="0 0 ${footprint_vertical_offset}" rpy="${PI/2} 0 ${PI/2}"/>
@@ -112,5 +118,5 @@
   </link>
   <xacro:unless value="$(optenv JACKAL_FRONT_ACCESSORY_FENDER 0)">
-    <link name="front_fender_link">
+    <link name="$(arg ns)front_fender_link">
       <visual>
         <geometry>
@@ -122,5 +128,5 @@
   </xacro:unless>
   <xacro:if value="$(optenv JACKAL_FRONT_ACCESSORY_FENDER 0)">
-    <link name="front_fender_link">
+    <link name="$(arg ns)front_fender_link">
       <visual>
         <geometry>
@@ -130,18 +136,18 @@
       </visual>
     </link>
-    <link name="front_fender_accessory_link"/>
+    <link name="$(arg ns)front_fender_accessory_link"/>
     <joint name="front_fender_accessory_joint" type="fixed">
       <origin xyz="0.25629 0 0.07455" rpy="${PI} 0 0" />
-      <parent link="front_fender_link" />
-      <child link="front_fender_accessory_link" />
+      <parent link="$(arg ns)front_fender_link" />
+      <child link="$(arg ns)front_fender_accessory_link" />
     </joint>
   </xacro:if>
-  <joint name="front_fender_joint" type="fixed">
+  <joint name="$(arg ns)front_fender_joint" type="fixed">
     <origin xyz="0 0 0" rpy="0 0 0"/>
-    <parent link="chassis_link" />
-    <child link="front_fender_link" />
+    <parent link="$(arg ns)chassis_link" />
+    <child link="$(arg ns)front_fender_link" />
   </joint>
   <xacro:unless value="$(optenv JACKAL_REAR_ACCESSORY_FENDER 0)">
-    <link name="rear_fender_link">
+    <link name="$(arg ns)rear_fender_link">
       <visual>
         <geometry>
@@ -153,5 +159,5 @@
   </xacro:unless>
   <xacro:if value="$(optenv JACKAL_REAR_ACCESSORY_FENDER 0)">
-    <link name="rear_fender_link">
+    <link name="$(arg ns)rear_fender_link">
       <visual>
         <geometry>
@@ -161,18 +167,18 @@
       </visual>
     </link>
-    <link name="rear_fender_accessory_link"/>
+    <link name="$(arg ns)rear_fender_accessory_link"/>
     <joint name="rear_fender_accessory_joint" type="fixed">
       <origin xyz="0.25629 0 0.07455" rpy="${PI} 0 0" />
-      <parent link="rear_fender_link" />
-      <child link="rear_fender_accessory_link" />
+      <parent link="$(arg ns)rear_fender_link" />
+      <child link="$(arg ns)rear_fender_accessory_link" />
     </joint>
   </xacro:if>
   <joint name="rear_fender_joint" type="fixed">
     <origin xyz="0 0 0" rpy="0 0 ${PI}"/>
-    <parent link="chassis_link" />
-    <child link="rear_fender_link" />
+    <parent link="$(arg ns)chassis_link" />
+    <child link="$(arg ns)rear_fender_link" />
   </joint>
   <!-- IMU LINK -->
-  <link name="imu_link">
+  <link name="$(arg ns)imu_link">
     <inertial>
       <mass value="0.001"/>
@@ -183,9 +189,9 @@
   <joint name="imu_joint" type="fixed">
     <origin xyz="0 0 0" rpy="0 0 0" />
-    <parent link="base_link" />
-    <child link="imu_link" />
+    <parent link="$(arg ns)base_link" />
+    <child link="$(arg ns)imu_link" />
   </joint>
   <!-- TODO: Same note as applies to imu_link -->
-  <link name="navsat_link">
+  <link name="$(arg ns)navsat_link">
     <visual>
       <geometry>
@@ -197,38 +203,70 @@
   </link>
   <joint name="navsat_joint" type="fixed">
-    <parent link="chassis_link" />
-    <child link="navsat_link" />
+    <parent link="$(arg ns)chassis_link" />
+    <child link="$(arg ns)navsat_link" />
     <origin xyz="-0.180 0.126 0.1815" />
   </joint>
-  <link name="mid_mount"></link>
+  <link name="$(arg ns)mid_mount"></link>
   <joint name="mid_mount_joint" type="fixed">
-    <parent link="chassis_link" />
-    <child link="mid_mount" />
+    <parent link="$(arg ns)chassis_link" />
+    <child link="$(arg ns)mid_mount" />
     <origin xyz="0 0 ${chassis_height}" />
   </joint>
-  <link name="rear_mount"></link>
+  <link name="$(arg ns)rear_mount"></link>
   <joint name="rear_mount_joint" type="fixed">
-    <parent link="mid_mount" />
-    <child link="rear_mount" />
+    <parent link="$(arg ns)mid_mount" />
+    <child link="$(arg ns)rear_mount" />
     <origin xyz="${-mount_spacing} 0 0" />
   </joint>
-  <link name="front_mount"></link>
+  <link name="$(arg ns)front_mount"></link>
   <joint name="front_mount_joint" type="fixed">
-    <parent link="mid_mount" />
-    <child link="front_mount" />
+    <parent link="$(arg ns)mid_mount" />
+    <child link="$(arg ns)front_mount" />
     <origin xyz="${mount_spacing} 0 0" />
   </joint>
+  <material name="Red">
+      <color rgba="${255/255} ${0/255} ${0/255} 1.0"/>
+  </material>
+  <material name="Green">
+      <color rgba="${0/255} ${255/255} ${0/255} 1.0"/>
+  </material>
+  <material name="Blue">
+      <color rgba="${0/255} ${0/255} ${255/255} 1.0"/>
+  </material>
+  <!-- -->
+  <link name="$(arg ns)right_tag">
+      <inertial>
+          <origin xyz="0 0 0.184" rpy="-1.57 0 -1.57"/>
+          <mass value="0.1" />
+          <inertia ixx="1.0" ixy="0.0" ixz="0.0" iyy="1.0" iyz="0.0" izz="1.0" />
+      </inertial>
+      <collision>
+          <origin xyz="0 0 0.184" rpy="-1.57 0 -1.57"/>
+          <geometry>
+              <box size="0.05 0.026 0.102"/>
+          </geometry>
+      </collision>
+      <visual>
+          <origin xyz="0 0 0.184" rpy="-1.57 0 -1.57"/>
+          <geometry>
+              <mesh filename="package://jackal_custom/models/DecaWave/meshes/Decawave.stl"/>
+          </geometry>
+          <material name="Blue"/>
+      </visual>
+  </link>
+  <joint name="right_tag_joint" type="fixed">
+      <parent link="$(arg ns)chassis_link"/>
+      <child link="$(arg ns)right_tag"/>
+  </joint>
   <!-- Bring in simulation data for Gazebo. -->
-  <xacro:include filename="$(find jackal_custom)/urdf/xacro/jackal.gazebo.xacro" />
-  <!-- Optional standard accessories, including their simulation data. The rendering
-       of these into the final description is controlled by optenv variables, which
-       default each one to off.-->
-  <!--xacro:include filename="$(find jackal_description)/urdf/accessories.urdf.xacro" /-->
-  <!---->
+  <gazebo>
+    <plugin name="gazebo_ros_control" filename="libgazebo_ros_control.so">
+    </plugin>
+  </gazebo>
   <gazebo>
       <plugin name="p3d_base_controller" filename="libgazebo_ros_p3d.so">
           <alwaysOn>true</alwaysOn>
           <updateRate>10.0</updateRate>
-          <bodyName>odom</bodyName>
+          <bodyName>$(arg ns)base_link</bodyName>
           <frameName>world</frameName>
           <topicName>ground_truth/state</topicName>
@@ -238,3 +276,41 @@
       </plugin>
   </gazebo>
+  <gazebo>
+    <plugin name="imu_controller" filename="libhector_gazebo_ros_imu.so">
+      <updateRate>10.0</updateRate>
+      <bodyName>$(arg ns)imu_link</bodyName>
+      <topicName>imu/data</topicName>
+      <accelDrift>0 0 0</accelDrift>
+      <accelGaussianNoise>0 0 0</accelGaussianNoise>
+      <rateDrift>0 0 0 </rateDrift>
+      <rateGaussianNoise>0 0 0 </rateGaussianNoise>
+      <headingDrift>0</headingDrift>
+      <headingGaussianNoise>0</headingGaussianNoise>
+    </plugin>
+  </gazebo>
+  <gazebo reference="$(arg ns)right_tag">
+      <material>Gazebo/White</material>
+  </gazebo>
+  <gazebo reference="$(arg ns)base_link">
+    <turnGravityOff>false</turnGravityOff>
+  </gazebo>
+  <gazebo reference="$(arg ns)chassis_link">
+    <material>Gazebo/DarkGrey</material>
+    <turnGravityOff>false</turnGravityOff>
+  </gazebo>
+  <gazebo reference="$(arg ns)imu_link">
+    <turnGravityOff>false</turnGravityOff>
+  </gazebo>
+  <gazebo reference="$(arg ns)navsat_link">
+    <material>Gazebo/DarkGrey</material>
+    <turnGravityOff>false</turnGravityOff>
+  </gazebo>
+  <gazebo reference="$(arg ns)front_fender_link">
+    <material>Gazebo/Green</material>
+    <turnGravityOff>false</turnGravityOff>
+  </gazebo>
+  <gazebo reference="$(arg ns)rear_fender_link">
+    <material>Gazebo/Red</material>
+    <turnGravityOff>false</turnGravityOff>
+  </gazebo>
 </robot>

Commit message: chore: tidy up

File: src/catkin_ws/src/jackal_custom/urdf/xacro/jackal_custom_base.urdf.xacro (robot description, xacro)
@@ -23,4 +23,13 @@
   <material name="yellow"><color rgba="0.8 0.8 0.0 1.0" /></material>
   <material name="black"><color rgba="0.15 0.15 0.15 1.0" /></material>
+  <material name="Red">
+      <color rgba="${255/255} ${0/255} ${0/255} 1.0"/>
+  </material>
+  <material name="Green">
+      <color rgba="${0/255} ${255/255} ${0/255} 1.0"/>
+  </material>
+  <material name="Blue">
+      <color rgba="${0/255} ${0/255} ${255/255} 1.0"/>
+  </material>
   <xacro:macro name="wheel" params="prefix *joint_pose">
     <link name="${prefix}_wheel_link">
@@ -63,5 +72,5 @@
     </joint>
     <!-- In reality, Jackal has only two motors, one per side. However, it's more
-         straightforward for Gazebo to simulate as if there's an actuator per wheel. -->
+        straightforward for Gazebo to simulate as if there's an actuator per wheel. -->
     <transmission name="${prefix}_wheel_trans">
       <type>transmission_interface/SimpleTransmission</type>
@@ -123,5 +132,5 @@
           <mesh filename="package://jackal_description/meshes/jackal-fender.stl"/>
         </geometry>
-        <material name="yellow" />
+        <material name="Green" />
       </visual>
     </link>
@@ -133,5 +142,5 @@
           <mesh filename="package://jackal_description/meshes/accessory_fender.stl"/>
         </geometry>
-        <material name="yellow" />
+        <material name="Green" />
       </visual>
     </link>
@@ -154,5 +163,5 @@
           <mesh filename="package://jackal_description/meshes/jackal-fender.stl"/>
         </geometry>
-        <material name="yellow" />
+        <material name="Red" />
       </visual>
     </link>
@@ -164,5 +173,5 @@
           <mesh filename="package://jackal_description/meshes/accessory_fender.stl"/>
         </geometry>
-        <material name="yellow" />
+        <material name="Red" />
       </visual>
     </link>
@@ -225,13 +234,4 @@
     <origin xyz="${mount_spacing} 0 0" />
   </joint>
-  <material name="Red">
-      <color rgba="${255/255} ${0/255} ${0/255} 1.0"/>
-  </material>
-  <material name="Green">
-      <color rgba="${0/255} ${255/255} ${0/255} 1.0"/>
-  </material>
-  <material name="Blue">
-      <color rgba="${0/255} ${0/255} ${255/255} 1.0"/>
-  </material>
   <!-- -->
   <link name="$(arg ns)right_tag">

Commit message: feat: working PF and absolute estimation

File: src/catkin_ws/src/jackal_custom/urdf/xacro/jackal_custom_base.urdf.xacro (robot description, xacro)
@@ -237,10 +237,10 @@
   <link name="$(arg ns)right_tag">
       <inertial>
-          <origin xyz="0 0 0.184" rpy="-1.57 0 -1.57"/>
+          <origin xyz="0 0 0" rpy="-1.57 0 -1.57"/>
           <mass value="0.1" />
           <inertia ixx="1.0" ixy="0.0" ixz="0.0" iyy="1.0" iyz="0.0" izz="1.0" />
       </inertial>
       <collision>
-          <origin xyz="0 0 0.184" rpy="-1.57 0 -1.57"/>
+          <origin xyz="0 0 0" rpy="-1.57 0 -1.57"/>
           <geometry>
               <box size="0.05 0.026 0.102"/>
@@ -248,5 +248,5 @@
       </collision>
       <visual>
-          <origin xyz="0 0 0.184" rpy="-1.57 0 -1.57"/>
+          <origin xyz="0 0 00" rpy="-1.57 0 -1.57"/>
           <geometry>
               <mesh filename="package://jackal_custom/models/DecaWave/meshes/Decawave.stl"/>
@@ -258,4 +258,5 @@
       <parent link="$(arg ns)chassis_link"/>
       <child link="$(arg ns)right_tag"/>
+      <origin xyz="0 0 0.184" rpy="0 0 0"/>
   </joint>
   <!-- Bring in simulation data for Gazebo. -->

Commit message: feat: working inter agents visualization

File: src/catkin_ws/src/jackal_custom/urdf/xacro/jackal_custom_base.urdf.xacro (robot description, xacro)
@@ -33,27 +33,4 @@
   </material>
   <xacro:macro name="wheel" params="prefix *joint_pose">
-    <link name="${prefix}_wheel_link">
-      <visual>
-        <origin xyz="0 0 0" rpy="${PI/2} 0 0"/>
-        <geometry>
-          <mesh filename="package://jackal_description/meshes/jackal-wheel.stl"/>
-        </geometry>
-        <material name="black" />
-      </visual>
-      <collision>
-        <origin xyz="0 0 0" rpy="${PI/2} 0 0"/>
-        <geometry>
-          <cylinder radius="${wheel_radius}" length="${wheel_width}"/>
-        </geometry>
-      </collision>
-      <inertial>
-        <origin xyz="0 0 0" rpy="0 0 0"/>
-        <mass value="0.477"/>
-        <inertia
-          ixx="0.0013" ixy="0" ixz="0"
-          iyy="0.0024" iyz="0"
-          izz="0.0013"/>
-      </inertial>
-    </link>
     <gazebo reference="${prefix}_wheel_link">
       <material>Gazebo/DarkGrey</material>
@@ -82,15 +59,38 @@
       </actuator>
     </transmission>
+    <link name="${prefix}_wheel_link">
+      <visual>
+        <origin xyz="0 0 0" rpy="${PI/2} 0 0"/>
+        <geometry>
+          <mesh filename="package://jackal_description/meshes/jackal-wheel.stl"/>
+        </geometry>
+        <material name="black" />
+      </visual>
+      <collision>
+        <origin xyz="0 0 0" rpy="${PI/2} 0 0"/>
+        <geometry>
+          <cylinder radius="${wheel_radius}" length="${wheel_width}"/>
+        </geometry>
+      </collision>
+      <inertial>
+        <origin xyz="0 0 0" rpy="0 0 0"/>
+        <mass value="0.477"/>
+        <inertia
+          ixx="0.0013" ixy="0" ixz="0"
+          iyy="0.0024" iyz="0"
+          izz="0.0013"/>
+      </inertial>
+    </link>
   </xacro:macro>
-  <xacro:wheel prefix="front_left">
+  <xacro:wheel prefix="$(arg ns)front_left">
     <origin xyz="${wheelbase/2} ${track/2} ${wheel_vertical_offset}" rpy="0 0 0" />
   </xacro:wheel>
-  <xacro:wheel prefix="front_right">
+  <xacro:wheel prefix="$(arg ns)front_right">
     <origin xyz="${wheelbase/2} ${-track/2} ${wheel_vertical_offset}" rpy="0 0 0" />
   </xacro:wheel>
-  <xacro:wheel prefix="rear_left">
+  <xacro:wheel prefix="$(arg ns)rear_left">
     <origin xyz="${-wheelbase/2} ${track/2} ${wheel_vertical_offset}" rpy="0 0 0" />
   </xacro:wheel>
-  <xacro:wheel prefix="rear_right">
+  <xacro:wheel prefix="$(arg ns)rear_right">
     <origin xyz="${-wheelbase/2} ${-track/2} ${wheel_vertical_offset}" rpy="0 0 0" />
   </xacro:wheel>
